File: KiCad/Coco2Composite.kicad_pcb (KiCad board)
At the start: 2 copper layers, 52 x 36.5 mm, 19 parts, among them J1 MA03-1, J2 MA05-1, J3 AUDIO_JACK_3.5MM_PTH, Q1 PN2907, Q2 2N2222, U1 MC1372

Commit message: moved ground pad to hopefully have it work as a support strut anchor point
Parts:
- PAD1: footprint TestPoint:TestPoint_THTPad_2.0x2.0mm_Drill1.0mm -> MountingHole:MountingHole_2.2mm_M2_DIN965_Pad
- moved PAD1 45.8 mm to (163.3, 106.6)
- moved C3 4.97 mm to (162.1, 101.4)
- moved R7 4.21 mm to (152.5, 110.7), turned to -90 degrees
- moved R8 4.06 mm to (162.1, 98.5)
- moved R5 2.83 mm to (148.9, 115.8)
Connections:
- net COMP_OUT renamed /COMP_OUT
- net Net-(C1-Pad2) renamed /CHROM_BALANCE
- net Net-(Q2-B) renamed /Q1_E
- net Net-(Q2-E) renamed /Q2_E
- net Net-(U1-CHROM_IN) renamed /CHROM_IN
- net Net-(U1-CHROM_MOD_OUT) renamed /CHROM_MOD_OUT
- net Net-(U1-COL_A_IN) renamed /PHI-A
- net Net-(U1-COL_B_IN) renamed /PHI-B
- net Net-(U1-COL_REF_IN) renamed /CHB
- net Net-(U1-LUM_IN) renamed /Y
- net Net-(U1-OSC_IN) renamed /CLK
- net Net-(U1-RF_OUT) renamed /RF_OUT
- net Net-(U1-RF_TANK_1) renamed /RF_TANK_1
- net Net-(U1-RF_TANK_2) renamed /RF_TANK_2
- net SND renamed /SND
- net SND_OUT renamed /SND_OUT
- J3 pad S: GND -> (no net)
- Q1 pad 1: VCC -> (no net)
- R3 pad 3: VCC -> (no net)
Routing:
- net /SND: track 27.4 -> 31.8 mm
- net /SND_OUT: track 23.7 -> 26.7 mm
- net /COMP_OUT: track 5.37 -> 7.26 mm
- net /Q2_E: track 29.6 -> 30.7 mm

Commit message: Minor tweaks
Parts:
- PAD1: footprint MountingHole:MountingHole_2.2mm_M2_DIN965_Pad -> MountingHole:MountingHole_3.7mm_Pad
- moved PAD1 0.20 mm to (163.5, 106.6)
- moved J3 0.05 mm to (163.5, 117.7)
Routing:
- net /SND_OUT: track 26.7 -> 29.4 mm
