File: KiCad-Horizontal/Coco2Composite.kicad_pcb (KiCad board)
At the start: 2 copper layers, 52 x 36.5 mm, 19 parts, among them J1 MA03-1, J2 MA05-1, J3 AUDIO_JACK_3.5MM_PTH, Q1 PN2907, Q2 2N2222, U1 MC1372

Commit message: Increased the footprint for the resistors since the one I picked was still too small
Parts:
- R1, R4, R5, R6, R7: footprint Resistor_THT:R_Axial_DIN0204_L3.6mm_D1.6mm_P5.08mm_Horizontal -> Resistor_THT:R_Axial_DIN0207_L6.3mm_D2.5mm_P7.62mm_Horizontal
- moved R6 2.57 mm to (156.7, 90.6)
- moved R4 2.53 mm to (151.1, 108.1)
- moved R5 2.53 mm to (148.9, 118.3)
Routing:
- net /SND: track 31.5 -> 32.8 mm
- net /COMP_OUT: track 7.26 -> 8.33 mm
