File: KiCad-Horizontal/Coco2Composite.kicad_sch (KiCad schematic)
At the start: 21 parts, among them J1 MA03-1, J2 MA05-1, J3 AUDIO_JACK_3.5MM_PTH, Q1 PN2907, Q2 2N2222, U1 MC1372

Commit message: Fixed the bypass cap on the schematic
Connections:
- net GND: now also C4.2
- net VCC: no longer C4.2
Changed lines of the file:
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@@
-	)
-	(junction
-		(at 142.24 125.73)
-		(diameter 0)
-		(color 0 0 0 0)
 	)
 	(junction
@@
 	(wire
 		(pts
-			(xy 142.24 120.65) (xy 142.24 125.73)
-		)
-		(stroke
-			(width 0.1524)
-			(type solid)
-		)
-	)
-	(wire
-		(pts
 			(xy 80.01 168.91) (xy 88.9 168.91)
 		)
@@
 	(wire
 		(pts
-			(xy 142.24 125.73) (xy 142.24 134.62)
+			(xy 142.24 120.65) (xy 142.24 134.62)
 		)
 		(stroke
@@
 		(pts
 			(xy 157.48 95.25) (xy 160.02 95.25)
-		)
-		(stroke
-			(width 0)
-			(type default)
-		)
-	)
-	(wire
-		(pts
-			(xy 142.24 125.73) (xy 146.05 125.73)
 		)
 		(stroke
@@
 					(unit 1)
 				)
+			)
+		)
+	)
+	(symbol
+		(lib_id "power:GND")
+		(at 146.05 125.73 0)
+		(unit 1)
+		(exclude_from_sim no)
+		(in_bom yes)
+		(on_board yes)
+		(dnp no)
+		(property "Reference" "#GND07"
+			(at 146.05 125.73 0)
+			(effects
+				(font
+					(size 1.27 1.27)
+				)
+				(hide yes)
+			)
+		)
+		(property "Value" "GND"
+			(at 143.764 130.302 0)
+			(effects
+				(font
+					(size 1.778 1.5113)
+				)
+				(justify left bottom)
+			)
+		)
+		(property "Footprint" ""
+			(at 146.05 125.73 0)
+			(effects
+				(font
+					(size 1.27 1.27)
+				)
+				(hide yes)
+			)
+		)
+		(property "Datasheet" ""
+			(at 146.05 125.73 0)
+			(effects
+				(font
+					(size 1.27 1.27)
+				)
+				(hide yes)
+			)
+		)
+		(property "Description" "Power symbol creates a global label with name \"GND\" , ground"
+			(at 146.05 125.73 0)
+			(effects
+				(font
+					(size 1.27 1.27)
+				)
+				(hide yes)
+			)
+		)
+		(pin "1"
+		)
+		(instances
+			(project "Coco2Composite"
+				(path "/10b578e1-d913-42e6-b9e5-398116858bd9"
+					(reference "#GND07")
+					(unit 1)
+				)
